Commit message: 修正robot的urdf文件bug

File: urdf/njust_v2_fixed.urdf (robot description, URDF)
Before this commit: robot njust_v2_fixed, 19 links, 18 joints
Links:
- link FL_calf: geometry collision mesh filename=package://lcm_tools/meshes/FL_calf.STL; visual mesh filename=package://lcm_tools/meshes/FL_calf.STL
- link FL_hip: geometry collision mesh filename=package://lcm_tools/meshes/FL_hip.STL; visual mesh filename=package://lcm_tools/meshes/FL_hip.STL
- link FL_thigh: geometry collision mesh filename=package://lcm_tools/meshes/FL_thigh.STL; visual mesh filename=package://lcm_tools/meshes/FL_thigh.STL
- link FL_wheel: geometry collision mesh filename=package://lcm_tools/meshes/FL_wheel.STL; visual mesh filename=package://lcm_tools/meshes/FL_wheel.STL
- link FR_calf: geometry collision mesh filename=package://lcm_tools/meshes/FR_calf.STL; visual mesh filename=package://lcm_tools/meshes/FR_calf.STL
- link FR_hip: geometry collision mesh filename=package://lcm_tools/meshes/FR_hip.STL; visual mesh filename=package://lcm_tools/meshes/FR_hip.STL
- link FR_thigh: geometry collision mesh filename=package://lcm_tools/meshes/FR_thigh.STL; visual mesh filename=package://lcm_tools/meshes/FR_thigh.STL
- link FR_wheel: geometry collision mesh filename=package://lcm_tools/meshes/FR_wheel.STL; visual mesh filename=package://lcm_tools/meshes/FR_wheel.STL
- link RL_calf: geometry collision mesh filename=package://lcm_tools/meshes/RL_calf.STL; visual mesh filename=package://lcm_tools/meshes/RL_calf.STL
- link RL_hip: geometry collision mesh filename=package://lcm_tools/meshes/RL_hip.STL; visual mesh filename=package://lcm_tools/meshes/RL_hip.STL
- link RL_thigh: geometry collision mesh filename=package://lcm_tools/meshes/RL_thigh.STL; visual mesh filename=package://lcm_tools/meshes/RL_thigh.STL
- link RL_wheel: geometry collision mesh filename=package://lcm_tools/meshes/RL_wheel.STL; visual mesh filename=package://lcm_tools/meshes/RL_wheel.STL
- link RR_calf: geometry collision mesh filename=package://lcm_tools/meshes/RR_calf.STL; visual mesh filename=package://lcm_tools/meshes/RR_calf.STL
- link RR_hip: geometry collision mesh filename=package://lcm_tools/meshes/RR_hip.STL; visual mesh filename=package://lcm_tools/meshes/RR_hip.STL
- link RR_thigh: geometry collision mesh filename=package://lcm_tools/meshes/RR_thigh.STL; visual mesh filename=package://lcm_tools/meshes/RR_thigh.STL
- link RR_wheel: geometry collision mesh filename=package://lcm_tools/meshes/RR_wheel.STL; visual mesh filename=package://lcm_tools/meshes/RR_wheel.STL
- link trunk: geometry collision mesh filename=package://lcm_tools/meshes/base_link.STL scale=1 1 1; visual mesh filename=package://lcm_tools/meshes/base_link.STL scale=1 1 1

File: urdf/njust_v2_wheel.urdf (robot description, URDF)
Before this commit: robot njust_v2_fixed, 19 links, 18 joints
Links:
- link FL_calf: geometry collision mesh filename=package://lcm_tools/meshes/FL_calf.STL; visual mesh filename=package://lcm_tools/meshes/FL_calf.STL
- link FL_hip: geometry collision mesh filename=package://lcm_tools/meshes/FL_hip.STL; visual mesh filename=package://lcm_tools/meshes/FL_hip.STL
- link FL_thigh: geometry collision mesh filename=package://lcm_tools/meshes/FL_thigh.STL; visual mesh filename=package://lcm_tools/meshes/FL_thigh.STL
- link FL_wheel: geometry collision mesh filename=package://lcm_tools/meshes/FL_wheel.STL; visual mesh filename=package://lcm_tools/meshes/FL_wheel.STL
- link FR_calf: geometry collision mesh filename=package://lcm_tools/meshes/FR_calf.STL; visual mesh filename=package://lcm_tools/meshes/FR_calf.STL
- link FR_hip: geometry collision mesh filename=package://lcm_tools/meshes/FR_hip.STL; visual mesh filename=package://lcm_tools/meshes/FR_hip.STL
- link FR_thigh: geometry collision mesh filename=package://lcm_tools/meshes/FR_thigh.STL; visual mesh filename=package://lcm_tools/meshes/FR_thigh.STL
- link FR_wheel: geometry collision mesh filename=package://lcm_tools/meshes/FR_wheel.STL; visual mesh filename=package://lcm_tools/meshes/FR_wheel.STL
- link RL_calf: geometry collision mesh filename=package://lcm_tools/meshes/RL_calf.STL; visual mesh filename=package://lcm_tools/meshes/RL_calf.STL
- link RL_hip: geometry collision mesh filename=package://lcm_tools/meshes/RL_hip.STL; visual mesh filename=package://lcm_tools/meshes/RL_hip.STL
- link RL_thigh: geometry collision mesh filename=package://lcm_tools/meshes/RL_thigh.STL; visual mesh filename=package://lcm_tools/meshes/RL_thigh.STL
- link RL_wheel: geometry collision mesh filename=package://lcm_tools/meshes/RL_wheel.STL; visual mesh filename=package://lcm_tools/meshes/RL_wheel.STL
- link RR_calf: geometry collision mesh filename=package://lcm_tools/meshes/RR_calf.STL; visual mesh filename=package://lcm_tools/meshes/RR_calf.STL
- link RR_hip: geometry collision mesh filename=package://lcm_tools/meshes/RR_hip.STL; visual mesh filename=package://lcm_tools/meshes/RR_hip.STL
- link RR_thigh: geometry collision mesh filename=package://lcm_tools/meshes/RR_thigh.STL; visual mesh filename=package://lcm_tools/meshes/RR_thigh.STL
- link RR_wheel: geometry collision mesh filename=package://lcm_tools/meshes/RR_wheel.STL; visual mesh filename=package://lcm_tools/meshes/RR_wheel.STL
- link trunk: geometry collision mesh filename=package://lcm_tools/meshes/base_link.STL scale=1 1 1; visual mesh filename=package://lcm_tools/meshes/base_link.STL scale=1 1 1

Commit message: 更新urdf的配置文件

File: urdf/njust_v2_fixed.urdf (robot description, URDF)
Before this commit: robot njust_v2_fixed, 19 links, 18 joints
Links:
- link FL_wheel: geometry collision mesh filename=package://lcm_tools/meshes/FL_wheel_B.STL; visual mesh filename=package://lcm_tools/meshes/FL_wheel_B.STL
- link FR_wheel: geometry collision mesh filename=package://lcm_tools/meshes/FR_wheel_B.STL; visual mesh filename=package://lcm_tools/meshes/FR_wheel_B.STL
- link RL_wheel: geometry collision mesh filename=package://lcm_tools/meshes/RL_wheel_B.STL; visual mesh filename=package://lcm_tools/meshes/RL_wheel_B.STL
- link RR_wheel: geometry collision mesh filename=package://lcm_tools/meshes/RR_wheel_B.STL; visual mesh filename=package://lcm_tools/meshes/RR_wheel_B.STL
- link trunk: geometry collision mesh filename=package://lcm_tools/meshes/base_link_sensors.STL scale=1 1 1; visual mesh filename=package://lcm_tools/meshes/base_link_sensors.STL scale=1 1 1

File: urdf/njust_v2_wheel.urdf (robot description, URDF)
Before this commit: robot njust_v2_fixed, 19 links, 18 joints
Links:
- link FL_wheel: geometry collision mesh filename=package://lcm_tools/meshes/FL_wheel_B.STL; visual mesh filename=package://lcm_tools/meshes/FL_wheel_B.STL
- link FR_wheel: geometry collision mesh filename=package://lcm_tools/meshes/FR_wheel_B.STL; visual mesh filename=package://lcm_tools/meshes/FR_wheel_B.STL
- link RL_wheel: geometry collision mesh filename=package://lcm_tools/meshes/RL_wheel_B.STL; visual mesh filename=package://lcm_tools/meshes/RL_wheel_B.STL
- link RR_wheel: geometry collision mesh filename=package://lcm_tools/meshes/RR_wheel_B.STL; visual mesh filename=package://lcm_tools/meshes/RR_wheel_B.STL
- link trunk: geometry collision mesh filename=package://lcm_tools/meshes/base_link_sensors.STL scale=1 1 1; visual mesh filename=package://lcm_tools/meshes/base_link_sensors.STL scale=1 1 1
